File: {{cookiecutter.repo_name}}/Hardware/{{cookiecutter.repo_name}}/{{cookiecutter.repo_name}}.kicad_sch (KiCad schematic)
At the start: 0 parts

Commit message: Boilerplate gitea
Other:
- company: {{cookiecutter.Institute}} -> {{cookiecutter.institute}}
Changed lines of the file:
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@@
     (title "{{cookiecutter.repo_name}}")
     (rev "${REVISION}")
-    (company "{{cookiecutter.Institute}}")
+    (company "{{cookiecutter.institute}}")
   )
   (sheet_instances
